File: simulation/kicad/simulation_schematic/pcb-001-ne555.kicad_sch (KiCad schematic)
At the start: 16 parts, among them J1 +5 V / GND power input, U1 NE555D

Commit message: docs: publish final PCB-001 engineering record
Changed lines of the file:
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@@
 			)
 		)
-		(property "Sim.Library" "C:\\Users\\avent\\OneDrive\\Documents\\pcb-001-ne555-astable-led-flasher\\kicad\\models\\uA555.sub"
+		(property "Sim.Library" "${KIPRJMOD}/../../../kicad/models/uA555.sub"
 			(at 170.18 102.87 0)
 			(hide yes)
@@
 		(unit 1)
 		(body_style 1)
-		(exclude_from_sim yes)
+		(exclude_from_sim no)
 		(in_bom yes)
 		(on_board yes)
@@
 		(in_pos_files yes)
 		(dnp no)
-		(fields_autoplaced yes)
 		(property "Reference" "RV1"
-			(at 107.9501 76.2 0)
+			(at 108.458 75.946 90)
 			(show_name no)
 			(do_not_autoplace no)
@@
 		)
 		(property "Value" "100 kOhm"
-			(at 105.4101 76.2 0)
+			(at 110.744 83.312 90)
 			(show_name no)
 			(do_not_autoplace no)
@@
 		(unit 1)
 		(body_style 1)
-		(exclude_from_sim yes)
+		(exclude_from_sim no)
 		(in_bom yes)
 		(on_board yes)
@@
 			(at 190.5 102.87 0)
 			(hide yes)
+			(show_name no)
+			(do_not_autoplace no)
+			(effects
+				(font
+					(size 1.27 1.27)
+				)
+			)
+		)
+		(property "Sim.Device" "D"
+			(at 190.5 102.87 0)
+			(hide yes)
+			(show_name no)
+			(do_not_autoplace no)
+			(effects
+				(font
+					(size 1.27 1.27)
+				)
+			)
+		)
+		(property "Sim.Params" "is=1e-18 rs=5 n=2"
+			(at 190.5 102.87 0)
+			(hide yes)
